Commit message: 超级左右互搏

File: rm_description/urdf/rm_75_right.urdf (robot description, URDF)
Before this commit: robot rm_75_description, 8 links, 7 joints
Links:
- removed link Link1
- removed link Link2
- removed link Link3
- removed link Link4
- removed link Link5
- removed link Link6
- removed link Link7
- removed link base_link
- added link right_Link1, mass 0.593563458735581; collision mesh filename=package://rm_description/meshes/rm_75_arm/link1.STL; visual mesh filename=package://rm_description/meshes/rm_75_arm/link1.STL
- added link right_Link2, mass 0.432849770310974; collision mesh filename=package://rm_description/meshes/rm_75_arm/link2.STL; visual mesh filename=package://rm_description/meshes/rm_75_arm/link2.STL
- added link right_Link3, mass 0.431325495678459; collision mesh filename=package://rm_description/meshes/rm_75_arm/link3.STL; visual mesh filename=package://rm_description/meshes/rm_75_arm/link3.STL
- added link right_Link4, mass 0.289633681619295; collision mesh filename=package://rm_description/meshes/rm_75_arm/link4.STL; visual mesh filename=package://rm_description/meshes/rm_75_arm/link4.STL
- added link right_Link5, mass 0.239419768320061; collision mesh filename=package://rm_description/meshes/rm_75_arm/link5.STL; visual mesh filename=package://rm_description/meshes/rm_75_arm/link5.STL
- added link right_Link6, mass 0.218799761431682; collision mesh filename=package://rm_description/meshes/rm_75_arm/link6.STL; visual mesh filename=package://rm_description/meshes/rm_75_arm/link6.STL
- added link right_Link7, mass 0.0649018034311231; collision mesh filename=package://rm_description/meshes/rm_75_arm/link7.STL; visual mesh filename=package://rm_description/meshes/rm_75_arm/link7.STL
- added link right_base_link, mass 0.841071174772543; collision mesh filename=package://rm_description/meshes/rm_75_arm/base_link.STL; visual mesh filename=package://rm_description/meshes/rm_75_arm/base_link.STL
Joints:
- removed joint joint1
- removed joint joint2
- removed joint joint3
- removed joint joint4
- removed joint joint5
- removed joint joint6
- removed joint joint7
- added joint right_joint1: type revolute, parent base_link, child Link1, origin xyz=0 0 0.2405 rpy=-1.5708 0 0, axis 0 -1 0, limit lower=-3.1 upper=3.1 effort=60 velocity=3.14
- added joint right_joint2: type revolute, parent Link1, child Link2, origin xyz=0 0 0 rpy=1.5708 0 0, axis 0 1 0, limit lower=-2.268 upper=2.268 effort=60 velocity=3.14
- added joint right_joint3: type revolute, parent Link2, child Link3, origin xyz=0 0 0.256 rpy=-1.5708 0 0, axis 0 -1 0, limit lower=-3.1 upper=3.1 effort=30 velocity=3.92
- added joint right_joint4: type revolute, parent Link3, child Link4, origin xyz=0 0 0 rpy=1.5708 0 0, axis 0 1 0, limit lower=-2.355 upper=2.355 effort=30 velocity=3.92
- added joint right_joint5: type revolute, parent Link4, child Link5, origin xyz=0 0 0.21 rpy=-1.5708 0 0, axis 0 -1 0, limit lower=-3.1 upper=3.1 effort=10 velocity=3.92
- added joint right_joint6: type revolute, parent Link5, child Link6, origin xyz=0 0 0 rpy=1.5708 0 0, axis 0 1 0, limit lower=-2.233 upper=2.233 effort=10 velocity=3.92
- added joint right_joint7: type revolute, parent Link6, child Link7, origin xyz=0 0 0.144 rpy=0 0 0, axis 0 0 1, limit lower=-6.28 upper=6.28 effort=10 velocity=3.92
