Commit message: 左臂 Moveit 节点成功

File: rm_description/urdf/rm_75_left.urdf (robot description, URDF)
Before this commit: robot rm_75_description_left, 8 links, 7 joints
Links:
- added link world
Joints:
- added joint left_base_mount: type fixed, parent world, child left_base_link, origin xyz=0.0 0.1 0.0 rpy=0.0 0.0 -0.7853981634
