Commit message: 完美双臂

File: rm_moveit2_config/rm_75_config/config/rm_75_description_dual.ros2_control.xacro (robot description, xacro)
@@ -2,5 +2,6 @@
 <robot xmlns:xacro="http://www.ros.org/wiki/xacro">
   <xacro:macro name="rm_75_description_ros2_control" params="name initial_positions_file">
-    <xacro:property name="initial_positions" value="${xacro.load_yaml(initial_positions_file)['initial_positions']}"/>
+    <xacro:property name="initial_positions"
+      value="${xacro.load_yaml(initial_positions_file)['initial_positions']}" />
     <ros2_control name="${name}" type="system">
       <hardware>
@@ -9,51 +10,51 @@
       </hardware>
       <joint name="left_joint1">
-        <command_interface name="position"/>
+        <command_interface name="position" />
         <state_interface name="position">
           <param name="initial_value">${initial_positions['left_joint1']}</param>
         </state_interface>
-        <state_interface name="velocity"/>
+        <state_interface name="velocity" />
       </joint>
       <joint name="left_joint2">
-        <command_interface name="position"/>
+        <command_interface name="position" />
         <state_interface name="position">
           <param name="initial_value">${initial_positions['left_joint2']}</param>
         </state_interface>
-        <state_interface name="velocity"/>
+        <state_interface name="velocity" />
       </joint>
       <joint name="left_joint3">
-        <command_interface name="position"/>
+        <command_interface name="position" />
         <state_interface name="position">
           <param name="initial_value">${initial_positions['left_joint3']}</param>
         </state_interface>
-        <state_interface name="velocity"/>
+        <state_interface name="velocity" />
       </joint>
       <joint name="left_joint4">
-        <command_interface name="position"/>
+        <command_interface name="position" />
         <state_interface name="position">
           <param name="initial_value">${initial_positions['left_joint4']}</param>
         </state_interface>
-        <state_interface name="velocity"/>
+        <state_interface name="velocity" />
       </joint>
       <joint name="left_joint5">
-        <command_interface name="position"/>
+        <command_interface name="position" />
         <state_interface name="position">
           <param name="initial_value">${initial_positions['left_joint5']}</param>
         </state_interface>
-        <state_interface name="velocity"/>
+        <state_interface name="velocity" />
       </joint>
       <joint name="left_joint6">
-        <command_interface name="position"/>
+        <command_interface name="position" />
         <state_interface name="position">
           <param name="initial_value">${initial_positions['left_joint6']}</param>
         </state_interface>
-        <state_interface name="velocity"/>
+        <state_interface name="velocity" />
       </joint>
       <joint name="left_joint7">
-        <command_interface name="position"/>
+        <command_interface name="position" />
         <state_interface name="position">
           <param name="initial_value">${initial_positions['left_joint7']}</param>
         </state_interface>
-        <state_interface name="velocity"/>
+        <state_interface name="velocity" />
       </joint>
     </ros2_control>
